File: doc/pcb/817.kicad_pcb (KiCad board)
At the start: 2 copper layers, 54.6 x 34.9 mm, 15 parts, among them J1 Conn_01x06_Male, J2 Conn_01x05_Male, K1 G5LE-1, K2 G5LE-1, Q1 S8050, Q2 S8050, U1 PC817

Commit message: Add files via upload
update pcb
Parts:
- Q1, Q2: value S8050 -> S8550
- R3, R4: value 1k -> 200
- moved Q1 3.32 mm to (156.7, 81.5), turned to 180 degrees
- moved Q2 2.95 mm to (162.7, 81.5), turned to 180 degrees
Connections:
- D1 pad 1: Net-(D1-Pad1) -> VDC
- D1 pad 2: GND -> Net-(D1-Pad2)
- D2 pad 1: Net-(D2-Pad1) -> VDC
- D2 pad 2: GND -> Net-(D2-Pad2)
- K1 pad 2: GND -> VDC
- K1 pad 5: Net-(D1-Pad1) -> Net-(D1-Pad2)
- K2 pad 2: GND -> VDC
- K2 pad 5: Net-(D2-Pad1) -> Net-(D2-Pad2)
- Q1 pad 1: Net-(D1-Pad1) -> Net-(D1-Pad2)
- Q1 pad 3: VDC -> GND
- Q2 pad 1: Net-(D2-Pad1) -> Net-(D2-Pad2)
- Q2 pad 3: VDC -> GND
Routing:
- net Net-(D2-Pad2): track 0.00 -> 82.7 mm
- net GND: track 98.9 -> 31.0 mm
- net Net-(D2-Pad1): track 59.9 -> 0.00 mm
- net Net-(D1-Pad2): track 0.00 -> 53.8 mm
- net Net-(D1-Pad1): track 41.9 -> 0.00 mm
- net VDC: track 53.2 -> 89.8 mm
- net Net-(Q1-Pad2): track 9.27 -> 8.57 mm
Other:
- board text added: "3.3v"
- board text removed: "5v"
